Commit message: interface changes

File: config/lexus_model.urdf (robot description, URDF)
Before this commit: robot lexus, 2 links, 1 joints
Links:
- link lexus_model: geometry visual mesh filename=package://multi_angle_interface/config/lexus_meshes/dae/Ext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 scale=1.0 1.02346 1.041
Joints:
- joint link_BaseLink: origin xyz=-0.05 0 -0.60 rpy=0 0 1.5708 -> xyz=-0.05 0 -1.80 rpy=0 0 1.5708
